File: src/PCB/ControlBoard/ControlBoard.kicad_pcb (KiCad board)
At the start: 2 copper layers, 76 x 76 mm, 32 parts, among them J1 Power, J2 OLED, J3 RGBW Control, SW1 Button, SW2 Button, SW3 Button, SW4 Button, SW5 Button, U1 LMR51430, U2 XIAO-RP2040-SMD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

Commit message: Finalise PCB and upload gerbers
Parts:
- added G***: LOGO, LOGO, F.Cu at (81.2, 68.0)
- added G***: LOGO, LOGO, F.Cu at (57.0, 67.5)
- added G***: LOGO, LOGO, F.Cu at (86.2, 76.5)
- added G***: LOGO, LOGO, F.Cu at (68.4, 58.1)
- added G***: LOGO, LOGO, F.Cu at (86.2, 69.3)
Routing:
- net GND: vias 60 -> 20
