File: src/PCB/VideographyLight/VideographyLight.kicad_pcb (KiCad board)
At the start: 2 copper layers, 100 x 100 mm, 4 parts

Commit message: Upload Light PCB
Parts:
- added C1: 10μF, Capacitor_SMD:C_1210_3225Metric_Pad1.33x2.70mm_HandSolder, F.Cu at (31.3, 93.4)
- added C10: 10μF, Capacitor_SMD:C_1210_3225Metric_Pad1.33x2.70mm_HandSolder, F.Cu at (97.9, 104.3)
- added C11: 10μF, Capacitor_SMD:C_1210_3225Metric_Pad1.33x2.70mm_HandSolder, F.Cu at (97.1, 91.0)
- added C2: 10μF, Capacitor_SMD:C_1210_3225Metric_Pad1.33x2.70mm_HandSolder, F.Cu at (27.2, 105.9)
- added C3: 10μF, Capacitor_SMD:C_1210_3225Metric_Pad1.33x2.70mm_HandSolder, F.Cu at (49.8, 105.8)
- added C4: 10μF, Capacitor_SMD:C_1210_3225Metric_Pad1.33x2.70mm_HandSolder, F.Cu at (53.0, 93.2)
- added C5: 10μF, Capacitor_SMD:C_1210_3225Metric_Pad1.33x2.70mm_HandSolder, F.Cu at (50.4, 84.4)
- added C6: 10μF, Capacitor_SMD:C_1210_3225Metric_Pad1.33x2.70mm_HandSolder, F.Cu at (78.8, 116.5)
- added C7: 10μF, Capacitor_SMD:C_1210_3225Metric_Pad1.33x2.70mm_HandSolder, F.Cu at (82.2, 104.0)
- added C8: 10μF, Capacitor_SMD:C_1210_3225Metric_Pad1.33x2.70mm_HandSolder, F.Cu at (72.9, 94.7)
- added C9: 10μF, Capacitor_SMD:C_1210_3225Metric_Pad1.33x2.70mm_HandSolder, F.Cu at (97.4, 116.8)
- added D1: SS1H10-E3/61T, footprints:DIOM5127X229N, F.Cu at (32.1, 84.0)
- added D10: SS1H10-E3/61T, footprints:DIOM5127X229N, F.Cu at (103.0, 102.1)
- added D11: SS1H10-E3/61T, footprints:DIOM5127X229N, F.Cu at (102.7, 115.9)
- added D2: SS1H10-E3/61T, footprints:DIOM5127X229N, F.Cu at (32.2, 96.7)
- added D3: SS1H10-E3/61T, footprints:DIOM5127X229N, F.Cu at (54.0, 96.6)
- added D4: SS1H10-E3/61T, footprints:DIOM5127X229N, F.Cu at (59.0, 87.8)
- added D5: SS1H10-E3/61T, footprints:DIOM5127X229N, F.Cu at (63.2, 84.4)
- added D6: SS1H10-E3/61T, footprints:DIOM5127X229N, F.Cu at (83.0, 107.4)
- added D7: SS1H10-E3/61T, footprints:DIOM5127X229N, F.Cu at (87.2, 100.6)
- added D8: SS1H10-E3/61T, footprints:DIOM5127X229N, F.Cu at (80.8, 84.0)
- added D9: SS1H10-E3/61T, footprints:DIOM5127X229N, F.Cu at (102.4, 88.7)
- added IC1: AL8862SP-13, footprints:SOIC127P600X163-9N, F.Cu at (28.1, 88.8)
- added IC10: AL8862SP-13, footprints:SOIC127P600X163-9N, F.Cu at (102.6, 97.7)
- added IC11: AL8862SP-13, footprints:SOIC127P600X163-9N, F.Cu at (102.4, 111.4)
- added IC2: AL8862SP-13, footprints:SOIC127P600X163-9N, F.Cu at (28.5, 101.5)
- added IC3: AL8862SP-13, footprints:SOIC127P600X163-9N, F.Cu at (51.0, 101.3)
- added IC4: AL8862SP-13, footprints:SOIC127P600X163-9N, F.Cu at (51.8, 88.8)
- added IC5: AL8862SP-13, footprints:SOIC127P600X163-9N, F.Cu at (51.6, 80.0)
- added IC6: AL8862SP-13, footprints:SOIC127P600X163-9N, F.Cu at (79.9, 112.0)
- added IC7: AL8862SP-13, footprints:SOIC127P600X163-9N, F.Cu at (79.8, 99.6)
- added IC8: AL8862SP-13, footprints:SOIC127P600X163-9N, F.Cu at (74.1, 90.3)
- added IC9: AL8862SP-13, footprints:SOIC127P600X163-9N, F.Cu at (102.7, 84.3)
- added J1: Power, TerminalBlock_Phoenix:TerminalBlock_Phoenix_MKDS-1,5-2-5.08_1x02_P5.08mm_Horizontal, F.Cu at (52.3, 114.0)
- added J2: RGBW Control, TerminalBlock_Phoenix:TerminalBlock_Phoenix_MKDS-1,5-4-5.08_1x04_P5.08mm_Horizontal, F.Cu at (30.4, 114.0)
- added L1: 100uH, footprints:INDPM120120X600N, B.Cu at (39.9, 87.8)
- added L10: 100uH, footprints:INDPM120120X600N, B.Cu at (111.8, 91.5)
- added L11: 100uH, footprints:INDPM120120X600N, B.Cu at (111.8, 105.5)
- added L2: 100uH, footprints:INDPM120120X600N, B.Cu at (39.7, 101.4)
- added L3: 100uH, footprints:INDPM120120X600N, B.Cu at (68.5, 111.8)
- added L4: 100uH, footprints:INDPM120120X600N, B.Cu at (62.0, 98.4)
- added L5: 100uH, footprints:INDPM120120X600N, B.Cu at (62.0, 85.2)
- added L6: 100uH, footprints:INDPM120120X600N, B.Cu at (90.6, 111.8)
- added L7: 100uH, footprints:INDPM120120X600N, B.Cu at (90.6, 98.6)
- added L8: 100uH, footprints:INDPM120120X600N, B.Cu at (90.6, 85.4)
- added L9: 100uH, footprints:INDPM120120X600N, B.Cu at (112.0, 77.8)
- added LED1: L1MC-RGB2290500MP0, footprints:L1MCRGB2290500MP0, F.Cu at (32.5, 68.7)
- added LED10: L1MC-RGB2290500MP0, footprints:L1MCRGB2290500MP0, F.Cu at (47.9, 50.2)
- added LED11: L1MC-RGB2290500MP0, footprints:L1MCRGB2290500MP0, F.Cu at (47.9, 58.3)
- added LED12: L1MC-RGB2290500MP0, footprints:L1MCRGB2290500MP0, F.Cu at (47.9, 66.4)
- added LED13: L1MC-RGB2290500MP0, footprints:L1MCRGB2290500MP0, F.Cu at (63.2, 68.2)
- added LED14: L1MC-RGB2290500MP0, footprints:L1MCRGB2290500MP0, F.Cu at (63.2, 60.1)
- added LED15: L1MC-RGB2290500MP0, footprints:L1MCRGB2290500MP0, F.Cu at (63.2, 52.0)
- added LED16: L1MC-RGB2290500MP0, footprints:L1MCRGB2290500MP0, F.Cu at (63.2, 43.9)
- added LED17: L1MC-RGB2290500MP0, footprints:L1MCRGB2290500MP0, F.Cu at (63.2, 35.8)
- added LED18: L1MC-RGB2290500MP0, footprints:L1MCRGB2290500MP0, F.Cu at (63.2, 27.7)
- added LED19: L1MC-RGB2290500MP0, footprints:L1MCRGB2290500MP0, F.Cu at (78.1, 26.0)
- added LED2: L1MC-RGB2290500MP0, footprints:L1MCRGB2290500MP0, F.Cu at (32.5, 60.6)
- added LED20: L1MC-RGB2290500MP0, footprints:L1MCRGB2290500MP0, F.Cu at (92.8, 67.8)
- added LED21: L1MC-RGB2290500MP0, footprints:L1MCRGB2290500MP0, F.Cu at (108.4, 26.3)
- added LED22: L1MC-RGB2290500MP0, footprints:L1MCRGB2290500MP0, F.Cu at (78.2, 34.1)
- added LED23: L1MC-RGB2290500MP0, footprints:L1MCRGB2290500MP0, F.Cu at (92.9, 59.7)
- added LED24: L1MC-RGB2290500MP0, footprints:L1MCRGB2290500MP0, F.Cu at (108.4, 34.2)
- added LED25: L1MC-RGB2290500MP0, footprints:L1MCRGB2290500MP0, F.Cu at (78.1, 42.4)
- added LED26: L1MC-RGB2290500MP0, footprints:L1MCRGB2290500MP0, F.Cu at (92.9, 51.7)
- added LED27: L1MC-RGB2290500MP0, footprints:L1MCRGB2290500MP0, F.Cu at (108.5, 42.0)
- added LED28: L1MC-RGB2290500MP0, footprints:L1MCRGB2290500MP0, F.Cu at (78.0, 50.6)
- added LED29: L1MC-RGB2290500MP0, footprints:L1MCRGB2290500MP0, F.Cu at (93.1, 43.7)
- added LED3: L1MC-RGB2290500MP0, footprints:L1MCRGB2290500MP0, F.Cu at (32.5, 52.5)
- added LED30: L1MC-RGB2290500MP0, footprints:L1MCRGB2290500MP0, F.Cu at (108.5, 49.8)
- added LED31: L1MC-RGB2290500MP0, footprints:L1MCRGB2290500MP0, F.Cu at (78.1, 58.6)
- added LED32: L1MC-RGB2290500MP0, footprints:L1MCRGB2290500MP0, F.Cu at (93.2, 35.9)
- added LED33: L1MC-RGB2290500MP0, footprints:L1MCRGB2290500MP0, F.Cu at (108.5, 57.6)
- added LED34: L1MC-RGB2290500MP0, footprints:L1MCRGB2290500MP0, F.Cu at (78.0, 66.6)
- added LED35: L1MC-RGB2290500MP0, footprints:L1MCRGB2290500MP0, F.Cu at (93.4, 27.9)
- added LED36: L1MC-RGB2290500MP0, footprints:L1MCRGB2290500MP0, F.Cu at (108.3, 65.6)
- added LED4: L1MC-RGB2290500MP0, footprints:L1MCRGB2290500MP0, F.Cu at (32.5, 44.4)
- added LED5: L1MC-RGB2290500MP0, footprints:L1MCRGB2290500MP0, F.Cu at (32.5, 36.3)
- added LED6: L1MC-RGB2290500MP0, footprints:L1MCRGB2290500MP0, F.Cu at (32.5, 28.2)
- added LED7: L1MC-RGB2290500MP0, footprints:L1MCRGB2290500MP0, F.Cu at (47.9, 25.9)
- added LED8: L1MC-RGB2290500MP0, footprints:L1MCRGB2290500MP0, F.Cu at (47.9, 34.0)
- added LED9: L1MC-RGB2290500MP0, footprints:L1MCRGB2290500MP0, F.Cu at (47.9, 42.1)
- added R1: 0.5Ω, Resistor_SMD:R_2010_5025Metric_Pad1.40x2.65mm_HandSolder, F.Cu at (25.6, 82.6)
- added R10: 0.5Ω, Resistor_SMD:R_2010_5025Metric_Pad1.40x2.65mm_HandSolder, F.Cu at (97.2, 98.3)
- added R11: 0.5Ω, Resistor_SMD:R_2010_5025Metric_Pad1.40x2.65mm_HandSolder, F.Cu at (97.0, 110.8)
- added R2: 0.5Ω, Resistor_SMD:R_2010_5025Metric_Pad1.40x2.65mm_HandSolder, F.Cu at (26.9, 95.2)
- added R3: 0.5Ω, Resistor_SMD:R_2010_5025Metric_Pad1.40x2.65mm_HandSolder, F.Cu at (48.8, 95.0)
- added R4: 0.5Ω, Resistor_SMD:R_2010_5025Metric_Pad1.40x2.65mm_HandSolder, F.Cu at (56.4, 84.4)
- added R5: 0.5Ω, Resistor_SMD:R_2010_5025Metric_Pad1.40x2.65mm_HandSolder, F.Cu at (59.0, 80.4)
- added R6: 0.5Ω, Resistor_SMD:R_2010_5025Metric_Pad1.40x2.65mm_HandSolder, F.Cu at (77.8, 105.8)
- added R7: 0.5Ω, Resistor_SMD:R_2010_5025Metric_Pad1.40x2.65mm_HandSolder, F.Cu at (72.6, 101.4)
- added R8: 0.5Ω, Resistor_SMD:R_2010_5025Metric_Pad1.40x2.65mm_HandSolder, F.Cu at (73.9, 84.8)
- added R9: 0.5Ω, Resistor_SMD:R_2010_5025Metric_Pad1.40x2.65mm_HandSolder, F.Cu at (97.1, 85.0)
Routing:
- net 48V: track 0.00 -> 381.6 mm, vias 0 -> 9
- net Red_K_2: track 0.00 -> 130.8 mm, vias 0 -> 1
- net Red_A_2: track 0.00 -> 116.4 mm, vias 0 -> 2
- net WHITE_Control: track 0.00 -> 109.1 mm, vias 0 -> 1
- net GND: track 0.00 -> 106.7 mm, vias 0 -> 111
- net White_K_1: track 0.00 -> 98.9 mm, vias 0 -> 3
- net Blue_K_1: track 0.00 -> 81.5 mm, vias 0 -> 1
- net BLUE_Control: track 0.00 -> 75.7 mm, vias 0 -> 3
- net Blue_A_1: track 0.00 -> 73.9 mm, vias 0 -> 2
- net Red_K_1: track 0.00 -> 72.8 mm, vias 0 -> 3
- net White_A_1: track 0.00 -> 71.0 mm, vias 0 -> 2
- net White_K_2: track 0.00 -> 67.5 mm, vias 0 -> 1
- net Green_K_3: track 0.00 -> 59.9 mm, vias 0 -> 3
- net White_A_2: track 0.00 -> 57.6 mm, vias 0 -> 4
- net Green_K_1: track 0.00 -> 57.3 mm, vias 0 -> 1
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- added copper zone on B.Cu, net GND
- added copper zone on F.Cu, net GND
