File: src/PCB/VideographyLight/VideographyLight.kicad_sch (KiCad schematic)
At the start: 91 parts, among them IC1 AL8862SP-13, IC10 AL8862SP-13, IC11 AL8862SP-13, IC2 AL8862SP-13, IC3 AL8862SP-13, IC4 AL8862SP-13, IC5 AL8862SP-13, IC6 AL8862SP-13, IC7 AL8862SP-13, IC8 AL8862SP-13, IC9 AL8862SP-13

Commit message: Push model for CAD
Parts:
- added J1: Power, TerminalBlock_Phoenix:TerminalBlock_Phoenix_MKDS-1,5-2-5.08_1x02_P5.08mm_Horizontal, symbol Connector:Conn_01x02_Socket
- added J2: RGBW Control, TerminalBlock_Phoenix:TerminalBlock_Phoenix_MKDS-1,5-4-5.08_1x04_P5.08mm_Horizontal, symbol Connector:Conn_01x04_Socket
Connections:
- net 48V: now also J1.1 (Pin_1)
- net BLUE_Control: now also J2.3 (Pin_3)
- net GND: now also J1.2 (Pin_2)
- net GREEN_Control: now also J2.2 (Pin_2)
- net RED_Control: now also J2.1 (Pin_1)
- net WHITE_Control: now also J2.4 (Pin_4)

Commit message: Upload Light PCB
Parts:
- C1, C10, C11, C2, C3, C4, C5, C6, C7, C8, C9: footprint (none) -> Capacitor_SMD:C_1210_3225Metric_Pad1.33x2.70mm_HandSolder; Mouser Part Number (none) -> 81-GRM32EC72A106ME5K
- IC1, IC10, IC11, IC2, IC3, IC4, IC5, IC6, IC7, IC8, IC9: Mouser Price/Stock (none) -> https://www.mouser.co.uk/ProductDetail/Diodes-Incorporated/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
- R1, R10, R11, R2, R3, R4, R5, R6, R7, R8, R9: footprint (none) -> Resistor_SMD:R_2010_5025Metric_Pad1.40x2.65mm_HandSolder; Mouser Part Number (none) -> 71-WSLT2010R5000FEA1
Connections:
- net Cont_14 is gone; now on net Cont_13: LED21.7 (A_WHITE)
- net Cont_11: now also LED21.1 (A_BLUE)
- net Cont_12: now also LED21.5 (A_GREEN); no longer LED21.1 (A_BLUE)
- net Cont_13: no longer LED21.5 (A_GREEN)
- removed net A_RED_2: IC1.1 (SET), IC2.1 (SET), LED1.3 (A_RED), LED1.4 (K_RED), LED1.9 (A_RED_2), LED10.3 (A_RED), LED10.4 (K_RED), LED10.9 (A_RED_2), LED11.3 (A_RED), LED11.4 (K_RED), LED11.9 (A_RED_2), LED12.3 (A_RED), LED12.4 (K_RED), LED12.9 (A_RED_2), LED13.3 (A_RED), LED13.4 (K_RED), LED13.9 (A_RED_2), LED14.3 (A_RED), LED14.4 (K_RED), LED14.9 (A_RED_2), LED15.3 (A_RED), LED15.4 (K_RED), LED15.9 (A_RED_2), LED16.3 (A_RED), LED16.4 (K_RED), LED16.9 (A_RED_2), LED17.3 (A_RED), LED17.4 (K_RED), LED17.9 (A_RED_2), LED18.3 (A_RED), LED18.9 (A_RED_2), LED19.3 (A_RED), LED19.4 (K_RED), LED19.9 (A_RED_2), LED2.3 (A_RED), LED2.4 (K_RED), LED2.9 (A_RED_2), LED20.3 (A_RED), LED20.4 (K_RED), LED20.9 (A_RED_2), LED21.3 (A_RED), LED21.4 (K_RED), LED21.9 (A_RED_2), LED22.3 (A_RED), LED22.4 (K_RED), LED22.9 (A_RED_2), LED23.3 (A_RED), LED23.4 (K_RED), LED23.9 (A_RED_2), LED24.3 (A_RED), LED24.4 (K_RED), LED24.9 (A_RED_2), LED25.3 (A_RED), LED25.4 (K_RED), LED25.9 (A_RED_2), LED26.3 (A_RED), LED26.4 (K_RED), LED26.9 (A_RED_2), LED27.3 (A_RED), LED27.4 (K_RED), LED27.9 (A_RED_2), LED28.3 (A_RED), LED28.4 (K_RED), LED28.9 (A_RED_2), LED29.3 (A_RED), LED29.4 (K_RED), LED29.9 (A_RED_2), LED3.3 (A_RED), LED3.4 (K_RED), LED3.9 (A_RED_2), LED30.3 (A_RED), LED30.4 (K_RED), LED30.9 (A_RED_2), LED31.3 (A_RED), LED31.4 (K_RED), LED31.9 (A_RED_2), LED32.3 (A_RED), LED32.4 (K_RED), LED32.9 (A_RED_2), LED33.3 (A_RED), LED33.4 (K_RED), LED33.9 (A_RED_2), LED34.3 (A_RED), LED34.4 (K_RED), LED34.9 (A_RED_2), LED35.3 (A_RED), LED35.4 (K_RED), LED35.9 (A_RED_2), LED36.3 (A_RED), LED36.9 (A_RED_2), LED4.3 (A_RED), LED4.4 (K_RED), LED4.9 (A_RED_2), LED5.3 (A_RED), LED5.4 (K_RED), LED5.9 (A_RED_2), LED6.3 (A_RED), LED6.4 (K_RED), LED6.9 (A_RED_2), LED7.3 (A_RED), LED7.4 (K_RED), LED7.9 (A_RED_2), LED8.3 (A_RED), LED8.4 (K_RED), LED8.9 (A_RED_2), LED9.3 (A_RED), LED9.4 (K_RED), LED9.9 (A_RED_2), R1.1, R2.1
- new net: LED14.4 (K_RED), LED15.3 (A_RED), LED15.9 (A_RED_2)
- new net: LED15.4 (K_RED), LED16.3 (A_RED), LED16.9 (A_RED_2)
- new net: LED29.4 (K_RED), LED32.3 (A_RED), LED32.9 (A_RED_2)
- new net: LED32.4 (K_RED), LED35.3 (A_RED), LED35.9 (A_RED_2)
- new net: LED4.4 (K_RED), LED5.3 (A_RED), LED5.9 (A_RED_2)
- new net: LED5.4 (K_RED), LED6.3 (A_RED), LED6.9 (A_RED_2)
- new net: LED8.4 (K_RED), LED9.3 (A_RED), LED9.9 (A_RED_2)
- new net: LED10.3 (A_RED), LED10.9 (A_RED_2), LED9.4 (K_RED)
- new net: LED21.4 (K_RED), LED24.3 (A_RED), LED24.9 (A_RED_2)
- new net: LED24.4 (K_RED), LED27.3 (A_RED), LED27.9 (A_RED_2)
- new net: LED28.4 (K_RED), LED31.3 (A_RED), LED31.9 (A_RED_2)
- new net: LED31.4 (K_RED), LED34.3 (A_RED), LED34.9 (A_RED_2)
- new net: LED26.4 (K_RED), LED29.3 (A_RED), LED29.9 (A_RED_2)
- new net: LED20.4 (K_RED), LED23.3 (A_RED), LED23.9 (A_RED_2)
- new net: LED1.4 (K_RED), LED2.3 (A_RED), LED2.9 (A_RED_2)
- new net: LED2.4 (K_RED), LED3.3 (A_RED), LED3.9 (A_RED_2)
- new net: LED22.4 (K_RED), LED25.3 (A_RED), LED25.9 (A_RED_2)
- new net: LED25.4 (K_RED), LED28.3 (A_RED), LED28.9 (A_RED_2)
- new net: LED16.4 (K_RED), LED17.3 (A_RED), LED17.9 (A_RED_2)
- new net: LED17.4 (K_RED), LED18.3 (A_RED), LED18.9 (A_RED_2)
- new net: LED13.4 (K_RED), LED14.3 (A_RED), LED14.9 (A_RED_2)
- new net: LED33.4 (K_RED), LED36.3 (A_RED), LED36.9 (A_RED_2)
- new net: LED27.4 (K_RED), LED30.3 (A_RED), LED30.9 (A_RED_2)
- new net: LED30.4 (K_RED), LED33.3 (A_RED), LED33.9 (A_RED_2)
- new net: LED11.4 (K_RED), LED12.3 (A_RED), LED12.9 (A_RED_2)
- new net: LED19.4 (K_RED), LED22.3 (A_RED), LED22.9 (A_RED_2)
- new net: LED23.4 (K_RED), LED26.3 (A_RED), LED26.9 (A_RED_2)
- new net: LED7.4 (K_RED), LED8.3 (A_RED), LED8.9 (A_RED_2)
- new net: LED3.4 (K_RED), LED4.3 (A_RED), LED4.9 (A_RED_2)
- new net: LED10.4 (K_RED), LED11.3 (A_RED), LED11.9 (A_RED_2)
- new net Cont_1: LED6.4 (K_RED), LED7.3 (A_RED), LED7.9 (A_RED_2)
- new net Cont_10: LED21.3 (A_RED), LED21.9 (A_RED_2), LED35.4 (K_RED)
- new net Cont_5: LED12.4 (K_RED), LED13.3 (A_RED), LED13.9 (A_RED_2)
- new net Cont_9: LED20.3 (A_RED), LED20.9 (A_RED_2), LED34.4 (K_RED)
- new net Red_A_1: IC1.1 (SET), LED1.3 (A_RED), LED1.9 (A_RED_2), R1.1
- new net Red_A_2: IC2.1 (SET), LED19.3 (A_RED), LED19.9 (A_RED_2), R2.1

Commit message: Finalise PCB and upload gerbers
Changed lines of the file:
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@@
 					(size 1.27 1.27)
 				)
+				(hide yes)
 			)
 		)
